Commit message: Push changs

File: husky_dual_ur5_description/urdf/husky_dual_ur5.urdf.xacro (robot description, xacro)
@@ -26,9 +26,10 @@
   <xacro:arg name="robot_namespace" default="/" />
   <xacro:arg name="urdf_extras" default="empty.urdf" />
+  `<xacro:arg name="transmission_hw_interface" default="hardware_interface/EffortJointInterface"/>
   <!-- Included URDF/XACRO Files -->
   <xacro:include filename="$(find husky_dual_ur5_description)/urdf/decorations.urdf.xacro" />
   <xacro:include filename="$(find husky_description)/urdf/wheel.urdf.xacro" />
   <xacro:include filename="$(find husky_description)/urdf/accessories/sick_lms1xx_mount.urdf.xacro"/>
-  <xacro:include filename="$(find ur_description)/urdf/ur5.urdf.xacro" />
+  <xacro:include filename="$(find ur_description)/urdf/ur5_d435.urdf.xacro" />
   <xacro:property name="M_PI" value="3.14159"/>
   <!-- Base Size -->
@@ -52,5 +53,5 @@
     </visual>
     <collision>
-      <origin xyz="${( husky_front_bumper_extend - husky_rear_bumper_extend ) / 2.0} 0 ${base_z_size/4}" rpy="0 0 0" />
+      <origin xyz="${( husky_front_bumper_extend - husky_rear_bumper_extend ) / 2.0} 0.0 ${base_z_size/4}" rpy="0 0 0" />
       <geometry>
         <box size="${ base_x_size + husky_front_bumper_extend + husky_rear_bumper_extend } ${base_y_size} ${base_z_size/2}"/>
@@ -74,11 +75,12 @@
   <link name="inertial_link">
     <inertial>
-      <mass value="46.034"/>
-      <origin xyz="-0.00065 -0.085 0.062" />
+      <mass value="46"/>
+      <origin xyz="-0.00065 0.0 0.1" />
+      <!--origin xyz="-0.05 0 0.17" /-->
       <inertia ixx="0.6022" ixy="-0.02364" ixz="-0.1197" iyy="1.7386" iyz="-0.001544" izz="2.0296" />
     </inertial>
   </link>
   <joint name="inertial_joint" type="fixed">
-    <origin xyz="0 0 0" rpy="0 0 0" />
+    <origin xyz="0 0 0.0" rpy="0 0.2 0" />
     <parent link="base_link" />
     <child link="inertial_link" />
